File: KiCAD/main/finals/rev 2.1/main.kicad_sch (KiCad schematic)
At the start: 49 parts, among them J1 USB_C_Receptacle_USB2.0_14P, J2 Conn_Coaxial, J3 Conn_01x07_Socket, SW1 SW_SPDT, U1 SX1262IMLTRT, U2 TP4056-42-ESOP8, U3 BGS12P2L, U4 ESP32-S3-MINI-1, U6 MIC5219-3.3YMM, U7 CH340X

Commit message: added a huge schematic overhaul
Parts:
- removed H1, H2: MountingHole_Pad, MountingHole:MountingHole_2.2mm_M2_DIN965_Pad_TopBottom, symbol Mechanical:MountingHole_Pad
- removed TP5, TP6, TP7, TP8: TestPoint, TestPoint:TestPoint_Pad_1.5x1.5mm, symbol Connector:TestPoint
Other:
- note removed: "DNP"
