File: KiCAD/main/finals/rev 2.1/main.kicad_pcb (KiCad board)
At the start: 2 copper layers, 21.9 x 63.9 mm, 42 parts, among them J1 USB_C_Receptacle_USB2.0_14P, J2 Conn_Coaxial, J3 Conn_01x07_Socket, SW1 SW_SPDT, U1 SX1262IMLTRT, U2 TP4056-42-ESOP8, U3 BGS12P2L, U4 ESP32-S3-MINI-1, U6 MIC5219-3.3YMM, U7 CH340X

Commit message: added a huge schematic overhaul
Parts:
- removed H1, H2: MountingHole_Pad, MountingHole:MountingHole_2.2mm_M2_DIN965_Pad_TopBottom
- added TP1: TestPoint, TestPoint:TestPoint_Pad_1.5x1.5mm, B.Cu at (104.6, 59.0)
- added TP2: TestPoint, TestPoint:TestPoint_Pad_1.5x1.5mm, B.Cu at (99.0, 63.2)
- added TP3: TestPoint, TestPoint:TestPoint_Pad_1.5x1.5mm, B.Cu at (95.2, 60.0)
- added TP4: TestPoint, TestPoint:TestPoint_Pad_1.5x1.5mm, B.Cu at (101.4, 54.2)
Routing:
- net TMS: track 0.00 -> 14.1 mm, vias 0 -> 1
- net TDI: track 0.00 -> 13.8 mm, vias 0 -> 1
- net TCK: track 0.00 -> 8.40 mm, vias 0 -> 1
- net TDO: track 0.00 -> 2.69 mm, vias 0 -> 1
- net V-: track 286.2 -> 285.2 mm

Commit message: Rev 3 done!
Routing:
- net USB_DATA+: track 8.10 -> 10.7 mm
- net USB_DATA-: track 10.5 -> 12.0 mm
Changed lines of the file:
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@@
 		(capping no)
 		(filling no)
+		(zone_defaults)
 		(pcbplotparams
 			(layerselection 0x00000000_00000000_55555555_5755f5ff)
@@
 	)
 	(segment
+		(start 92.388079 66.563079)
+		(end 93.251158 65.7)
+		(width 0.2)
+		(layer "F.Cu")
+		(net "V-")
+	)
+	(segment
 		(start 105.118748 46.05)
 		(end 105.451158 46.05)
@@
 	)
 	(via
-		(at 93.345 65.659)
+		(at 92.388079 66.563079)
 		(size 0.6)
 		(drill 0.3)
@@
 	)
 	(segment
-		(start 90.551 68.400158)
-		(end 93.251158 65.7)
-		(width 0.2)
-		(layer "B.Cu")
-		(net "V-")
-	)
-	(segment
 		(start 93.2 45.858658)
 		(end 91.555342 45.858658)
@@
 	)
 	(segment
+		(start 92.388079 66.563079)
+		(end 90.551 68.400158)
+		(width 0.2)
+		(layer "B.Cu")
+		(net "V-")
+	)
+	(segment
 		(start 95.25 78.613)
 		(end 95.25 84.963)
@@
 	)
 	(segment
-		(start 102.258748 85.97)
-		(end 101.991158 86.23759)
+		(start 102.951158 81.2)
+		(end 102.951158 80.345158)
 		(width 0.2)
 		(layer "F.Cu")
@@
 	)
 	(segment
-		(start 102.991158 86.23759)
-		(end 102.991158 86.845)
+		(start 102.991158 87.45241)
+		(end 102.723568 87.72)
 		(width 0.2)
 		(layer "F.Cu")
@@
 	)
 	(segment
-		(start 101.991158 86.23759)
-		(end 101.991158 86.845)
+		(start 102.723568 87.72)
+		(end 102.258748 87.72)
+		(width 0.2)
+		(layer "F.Cu")
+		(net "USB_DATA+")
+	)
+	(segment
+		(start 102.4636 80.264)
+		(end 102.4636 81.9912)
+		(width 0.2)
+		(layer "F.Cu")
+		(net "USB_DATA+")
+	)
+	(segment
+		(start 102.991158 86.845)
+		(end 102.991158 87.45241)
 		(width 0.2)
 		(layer "F.Cu")
@@
 	)
 	(segment
-		(start 102.723568 85.97)
-		(end 102.258748 85.97)
+		(start 102.258748 87.72)
+		(end 101.991158 87.45241)
+		(width 0.2)
+		(layer "F.Cu")
+		(net "USB_DATA+")
+	)
+	(segment
+		(start 102.5144 80.2132)
+		(end 102.4636 80.264)
+		(width 0.2)
+		(layer "F.Cu")
+		(net "USB_DATA+")
+	)
+	(segment
+		(start 101.991158 87.45241)
+		(end 101.991158 86.845)
+		(width 0.2)
+		(layer "F.Cu")
+		(net "USB_DATA+")
+	)
+	(segment
+		(start 102.991158 82.518758)
+		(end 102.991158 86.845)
+		(width 0.2)
+		(layer "F.Cu")
+		(net "USB_DATA+")
+	)
+	(segment
+		(start 102.951158 80.345158)
+		(end 102.8192 80.2132)
 		(width 0.2)
 		(layer "F.Cu")
@@
 	)
 	(segment
-		(start 102.991158 86.23759)
-		(end 102.723568 85.97)
+		(start 102.4636 81.9912)
+		(end 102.991158 82.518758)
 		(width 0.2)
 		(layer "F.Cu")
@@
 	)
 	(segment
-		(start 102.951158 86.805)
-		(end 102.951158 81.2)
+		(start 102.8192 80.2132)
+		(end 102.5144 80.2132)
 		(width 0.2)
 		(layer "F.Cu")
@@
 	)
 	(segment
-		(start 102.491158 87.45241)
-		(end 102.223568 87.72)
+		(start 102.223568 85.97)
+		(end 102.491158 86.23759)
 		(width 0.2)
 		(layer "F.Cu")
@@
 	)
 	(segment
-		(start 103.491158 87.45241)
-		(end 103.223568 87.72)
+		(start 101.758748 85.97)
+		(end 102.223568 85.97)
 		(width 0.2)
 		(layer "F.Cu")
@@
 	)
 	(segment
-		(start 101.758748 87.72)
-		(end 101.491158 87.45241)
+		(start 102.348714 79.8132)
+		(end 102.0636 80.098315)
 		(width 0.2)
 		(layer "F.Cu")
@@
 	)
 	(segment
-		(start 102.223568 87.72)
-		(end 101.758748 87.72)
+		(start 102.984885 79.8132)
+		(end 102.348714 79.8132)
+		(width 0.2)
+		(layer "F.Cu")
+		(net "USB_DATA-")
+	)
+	(segment
+		(start 102.491158 86.23759)
+		(end 102.491158 86.845)
+		(width 0.2)
+		(layer "F.Cu")
+		(net "USB_DATA-")
+	)
+	(segment
+		(start 103.451158 81.2)
+		(end 103.451158 80.279473)
 		(width 0.2)
 		(layer "F.Cu")
@@
 	)
 	(segment
-		(start 102.491158 86.845)
-		(end 102.491158 87.45241)
+		(start 101.491158 86.23759)
+		(end 101.758748 85.97)
 		(width 0.2)
 		(layer "F.Cu")
@@
 	)
 	(segment
-		(start 103.223568 87.72)
-		(end 101.758748 87.72)
+		(start 103.451158 80.279473)
+		(end 102.984885 79.8132)
 		(width 0.2)
 		(layer "F.Cu")
@@
 	)
 	(segment
-		(start 103.491158 86.845)
-		(end 103.491158 87.45241)
+		(start 101.491158 86.845)
+		(end 101.491158 86.23759)
 		(width 0.2)
 		(layer "F.Cu")
@@
 	)
 	(segment
-		(start 101.491158 87.45241)
-		(end 101.491158 86.845)
+		(start 102.0636 82.2008)
+		(end 102.491158 82.628358)
 		(width 0.2)
 		(layer "F.Cu")
@@
 	)
 	(segment
-		(start 103.451158 81.2)
-		(end 103.451158 86.805)
+		(start 102.491158 82.628358)
+		(end 102.491158 86.845)
+		(width 0.2)
+		(layer "F.Cu")
+		(net "USB_DATA-")
+	)
+	(segment
+		(start 102.0636 80.098315)
+		(end 102.0636 82.2008)
 		(width 0.2)
 		(layer "F.Cu")

Commit message: Brushing off dust
Parts:
- moved C5 0.11 mm to (101.3, 78.8)
- moved C15 0.10 mm to (100.9, 84.9)
Routing:
- net V-: track 285.2 -> 430.0 mm, vias 15 -> 16
- net VCC: track 118.4 -> 121.8 mm, vias 4 -> 7
- net Net-(D1-K): track 15.6 -> 18.8 mm
- net Net-(U1-VREG): track 6.07 -> 9.19 mm
- net Net-(U1-DCC_SW): track 7.56 -> 6.31 mm
- net V+: track 50.0 -> 49.4 mm
- added copper zone on B.Cu, net V-
