File: KiCAD/main/finals/rev2.1/main.kicad_pcb (KiCad board)
At the start: 2 copper layers, 30 x 65 mm, 47 parts, among them J1 USB_C_Receptacle_USB2.0_14P, J2 Conn_Coaxial, J3 Conn_01x07_Socket, SW1 SW_SPDT, U1 SX1262IMLTRT, U2 TP4056-42-ESOP8, U3 BGS12P2L, U4 ESP32-S3-MINI-1, U6 MIC5219-3.3YMM, U7 CH340X

Commit message: Replaced ESP-WROOM module with ESP32-S3 module for flexable usage and stocking
Parts:
- removed C18: 0.1uF, Capacitor_SMD:C_0402_1005Metric
- removed TP1, TP2, TP3, TP4: TestPoint, TestPoint:TestPoint_Pad_1.5x1.5mm
- removed U7: CH340X, Package_SO:MSOP-10_3x3mm_P0.5mm
- added C11: 0.1uF, Capacitor_SMD:C_0402_1005Metric, F.Cu at (103.9, 52.9)
- added C4: 0.1uF, Capacitor_SMD:C_0402_1005Metric, F.Cu at (115.3, 82.8)
- added D3: WS2812B, LED_SMD:LED_WS2812B_PLCC4_5.0x5.0mm_P3.2mm, F.Cu at (98.5, 71.8)
- added J4: Micro_SD_Card, customlib:SIM-SMD_8P-1040310811, B.Cu at (100.8, 48.9)
- added R10: 10K, Resistor_SMD:R_0603_1608Metric, F.Cu at (101.4, 59.7)
- added R11: 10K, Resistor_SMD:R_0603_1608Metric, B.Cu at (97.4, 48.9)
- added R12: 10K, Resistor_SMD:R_0603_1608Metric, B.Cu at (99.2, 47.8)
- added R13: 10K, Resistor_SMD:R_0603_1608Metric, B.Cu at (100.9, 46.5)
- added R4: 450R, Resistor_SMD:R_0402_1005Metric, F.Cu at (102.8, 74.9)
- added R5: 10K, Resistor_SMD:R_0603_1608Metric, B.Cu at (99.7, 52.7)
- added R8: 10K, Resistor_SMD:R_0603_1608Metric, B.Cu at (97.4, 52.2)
- added R9: 10K, Resistor_SMD:R_0603_1608Metric, F.Cu at (101.4, 63.4)
- added TCK1: TestPoint, TestPoint:TestPoint_Pad_1.5x1.5mm, B.Cu at (109.3, 66.8)
- added TDI1: TestPoint, TestPoint:TestPoint_Pad_1.5x1.5mm, B.Cu at (118.7, 65.8)
- added TDO1: TestPoint, TestPoint:TestPoint_Pad_1.5x1.5mm, B.Cu at (113.1, 70.0)
- added TMS1: TestPoint, TestPoint:TestPoint_Pad_1.5x1.5mm, B.Cu at (115.5, 61.0)
- added U2: CH340X, Package_SO:MSOP-10_3x3mm_P0.5mm, F.Cu at (118.0, 85.9)
- moved G*** 34.2 mm to (15.5, 15.3)
- renumbered C2 to C1, C12 to C10, C13 to C12, C7 to C13, C6 to C14, C10 to C15, C11 to C16, C14 to C17, C5 to C2, C1 to C3, C17 to C5, C15 to C6, C16 to C7, C4 to C8, C3 to C9, H1 to H2, H2 to H4, J3 to J1, J1 to J2, J2 to J3, L2 to L1, L1 to L2, R7 to R3, R5 to R6, R4 to R7, U6 to U1, U2 to U3, U3 to U5, U1 to U6
Connections:
- net Net-(SW1-A) renamed +5V
- net V- renamed GND
- C1 pad 2: VCC -> +3.3V
- C13 pad 1: VCC -> +3.3V
- C14 pad 1: VCC -> +3.3V
- C15 pad 1: VCC -> +3.3V
- C17 pad 2: VCC -> +3.3V
- C5 pad 2: VCC -> +3.3V
- C8 pad 2: VCC -> +3.3V
- C9 pad 2: VCC -> +3.3V
- J1 pad 2: VCC -> +3.3V
- R7 pad 1: VCC -> +3.3V
- U1 pad 3: VCC -> +3.3V
- U4 pad 16: unconnected-(U4-IO12-Pad16) -> DAT0
- U4 pad 17: unconnected-(U4-IO13-Pad17) -> DAT1
- U4 pad 18: unconnected-(U4-IO14-Pad18) -> CMD
- U4 pad 19: unconnected-(U4-IO15-Pad19) -> DAT3/CD
- U4 pad 20: ~{CHRG} -> DAT2
- U4 pad 21: ~{STDBY} -> CLK
- U4 pad 22: unconnected-(U4-IO18-Pad22) -> ~{CHRG}
- U4 pad 23: unconnected-(U4-USB_D--Pad23) -> ~{STDBY}
- U4 pad 3: VCC -> +3.3V
- U4 pad 44: unconnected-(U4-IO46-Pad44) -> NEOPXL_D
- U5 pad 4: VCC -> +3.3V
- U6 pad 1: VCC -> +3.3V
- U6 pad 10: VCC -> +3.3V
- U6 pad 11: VCC -> +3.3V
Routing:
- net +3.3V: track 0.00 -> 163.2 mm, vias 0 -> 8
- net VCC: track 121.8 -> 0.00 mm, vias 7 -> 0
- net DAT2: track 0.00 -> 52.4 mm, vias 0 -> 3
- net DAT3/CD: track 0.00 -> 43.2 mm, vias 0 -> 2
- net CMD: track 0.00 -> 34.6 mm, vias 0 -> 3
- net DAT1: track 0.00 -> 25.6 mm, vias 0 -> 1
- net DAT0: track 0.00 -> 22.9 mm, vias 0 -> 1
- net +5V: track 14.6 -> 36.6 mm, vias 0 -> 2
- net NEOPXL_D: track 0.00 -> 17.8 mm, vias 0 -> 2
- net GND: track 382.3 -> 397.4 mm
- net ~{CHRG}: track 28.7 -> 37.4 mm, vias 2 -> 4
- net ~{STDBY}: track 34.4 -> 42.8 mm
- net Net-(D3-DIN): track 0.00 -> 2.45 mm
- added copper zone on F.Cu, net GND
Other:
- board text added: "VIP(E)R Rev3"
- board text removed: "VIP(E)R Rev2.1"
- board text removed: "VIPR Rev2.1"
